Commit message: further modification

File: robot/hsr_mujoco/model/robot/hsrb4s/stl/hsrb4s.urdf (robot description, URDF)
Before this commit: robot hsrb, 46 links, 45 joints
Links:
- link arm_flex_link: geometry collision mesh filename=file:///home/akshay/Multiverse_hsr_robot/robot/hsr_mujoco/m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; visual mesh filename=file:///home/akshay/Multiverse_hsr_robot/robot/hsr_mujoco/m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
- link arm_lift_link: geometry collision mesh filename=file:///home/akshay/Multiverse_hsr_robot/robot/hsr_mujoco/m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; visual mesh filename=file:///home/akshay/Multiverse_hsr_robot/robot/hsr_mujoco/m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
- link arm_roll_link: geometry collision mesh filename=file:///home/akshay/Multiverse_hsr_robot/robot/hsr_mujoco/m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; visual mesh filename=file:///home/akshay/Multiverse_hsr_robot/robot/hsr_mujoco/m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
- link base_link: geometry collision mesh filename=file:///home/akshay/Multiverse_hsr_robot/robot/hsr_mujoco/m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; visual mesh filename=file:///home/akshay/Multiverse_hsr_robot/robot/hsr_mujoco/m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
- link base_range_sensor_link: geometry collision mesh filename=file:///home/akshay/Multiverse_hsr_robot/robot/hsr_mujoco/m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; visual mesh filename=file:///home/akshay/Multiverse_hsr_robot/robot/hsr_mujoco/m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
- link hand_l_distal_link: geometry collision mesh filename=file:///home/akshay/Multiverse_hsr_robot/robot/hsr_mujoco/m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; visual mesh filename=file:///home/akshay/Multiverse_hsr_robot/robot/hsr_mujoco/m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
- link hand_l_spring_proximal_link: geometry collision mesh filename=file:///home/akshay/Multiverse_hsr_robot/robot/hsr_mujoco/m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; visual mesh filename=file:///home/akshay/Multiverse_hsr_robot/robot/hsr_mujoco/m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
- link hand_palm_link: geometry collision mesh filename=file:///home/akshay/Multiverse_hsr_robot/robot/hsr_mujoco/m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; visual mesh filename=file:///home/akshay/Multiverse_hsr_robot/robot/hsr_mujoco/m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
- link hand_r_distal_link: geometry collision mesh filename=file:///home/akshay/Multiverse_hsr_robot/robot/hsr_mujoco/m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; visual mesh filename=file:///home/akshay/Multiverse_hsr_robot/robot/hsr_mujoco/m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
- link hand_r_spring_proximal_link: geometry collision mesh filename=file:///home/akshay/Multiverse_hsr_robot/robot/hsr_mujoco/m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; visual mesh filename=file:///home/akshay/Multiverse_hsr_robot/robot/hsr_mujoco/m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
- link head_l_stereo_camera_link: geometry visual mesh filename=file:///home/akshay/Multiverse_hsr_robot/robot/hsr_mujoco/m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
- link head_pan_link: geometry collision mesh filename=file:///home/akshay/Multiverse_hsr_robot/robot/hsr_mujoco/m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; visual mesh filename=file:///home/akshay/Multiverse_hsr_robot/robot/hsr_mujoco/m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
- link head_r_stereo_camera_link: geometry visual mesh filename=file:///home/akshay/Multiverse_hsr_robot/robot/hsr_mujoco/m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
- link head_rgbd_sensor_link: geometry collision mesh filename=file:///home/akshay/Multiverse_hsr_robot/robot/hsr_mujoco/m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; visual mesh filename=file:///home/akshay/Multiverse_hsr_robot/robot/hsr_mujoco/m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
- link head_tilt_link: geometry collision mesh filename=file:///home/akshay/Multiverse_hsr_robot/robot/hsr_mujoco/m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; collision mesh filename=file:///home/akshay/Multiverse_hsr_robot/robot/hsr_mujoco/m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
- link torso_lift_link: geometry collision mesh filename=file:///home/akshay/Multiverse_hsr_robot/robot/hsr_mujoco/m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; visual mesh filename=file:///home/akshay/Multiverse_hsr_robot/robot/hsr_mujoco/m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
- link wrist_flex_link: geometry collision cylinder length=0.04 radius=0.017; visual cylinder length=0.02 radius=0.017
- link wrist_roll_link: geometry collision mesh filename=file:///home/akshay/Multiverse_hsr_robot/robot/hsr_mujoco/m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; visual mesh filename=file:///home/akshay/Multiverse_hsr_robot/robot/hsr_mujoco/m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
