Commit message: restructure file system and added static transformation to stabilize rviz2

File: robot/hsr_description/robots/hsrb4s.obj.urdf (robot description, URDF)
Before this commit: robot hsrb, 46 links, 45 joints
Links:
- link arm_flex_link: geometry collision mesh filename=file://hsr_meshes/meshes/arm_v0/arm_flex.stl; visual mesh filename=file://hsr_meshes/meshes/arm_v0/arm_flex_light.obj
- link arm_lift_link: geometry collision mesh filename=file://hsr_meshes/meshes/arm_v0/shoulder.stl; visual mesh filename=file://hsr_meshes/meshes/arm_v0/shoulder.obj
- link arm_roll_link: geometry collision mesh filename=file://hsr_meshes/meshes/arm_v0/arm_roll.stl; visual mesh filename=file://hsr_meshes/meshes/arm_v0/arm_roll_light.obj
- link base_link: geometry collision mesh filename=file://hsr_meshes/meshes/base_v2/base.stl; visual mesh filename=file://hsr_meshes/meshes/base_v2/base_light.obj
- link base_range_sensor_link: geometry collision mesh filename=file://hsr_meshes/meshes/sensors/laser.stl; visual mesh filename=file://hsr_meshes/meshes/sensors/laser.obj
- link hand_l_distal_link: geometry collision mesh filename=file://hsr_meshes/meshes/hand_v0/l_distal.stl; visual mesh filename=file://hsr_meshes/meshes/hand_v0/l_distal.obj
- link hand_l_spring_proximal_link: geometry collision mesh filename=file://hsr_meshes/meshes/hand_v0/l_proximal.stl; visual mesh filename=file://hsr_meshes/meshes/hand_v0/l_proximal.obj
- link hand_palm_link: geometry collision mesh filename=file://hsr_meshes/meshes/hand_v0/palm.stl; visual mesh filename=file://hsr_meshes/meshes/hand_v0/palm.obj
- link hand_r_distal_link: geometry collision mesh filename=file://hsr_meshes/meshes/hand_v0/r_distal.stl; visual mesh filename=file://hsr_meshes/meshes/hand_v0/r_distal.obj
- link hand_r_spring_proximal_link: geometry collision mesh filename=file://hsr_meshes/meshes/hand_v0/r_proximal.stl; visual mesh filename=file://hsr_meshes/meshes/hand_v0/r_proximal.obj
- link head_l_stereo_camera_link: geometry visual mesh filename=file://hsr_meshes/meshes/sensors/head_camera.obj
- link head_pan_link: geometry collision mesh filename=file://hsr_meshes/meshes/head_v1/head_pan.stl; visual mesh filename=file://hsr_meshes/meshes/head_v1/head_pan.obj
- link head_r_stereo_camera_link: geometry visual mesh filename=file://hsr_meshes/meshes/sensors/head_camera.obj
- link head_rgbd_sensor_link: geometry collision mesh filename=file://hsr_meshes/meshes/sensors/rgbd.stl; visual mesh filename=file://hsr_meshes/meshes/sensors/rgbd_light.obj
- link head_tilt_link: geometry collision mesh filename=file://hsr_meshes/meshes/head_v1/head.stl; collision mesh filename=file://hsr_meshes/meshes/head_v1/tablet.stl
- link torso_lift_link: geometry collision mesh filename=file://hsr_meshes/meshes/torso_v0/torso.stl; visual mesh filename=file://hsr_meshes/meshes/torso_v0/torso_light.obj
- link wrist_flex_link: geometry collision cylinder length=0.04 radius=0.017; visual cylinder length=0.02 radius=0.017
- link wrist_roll_link: geometry collision mesh filename=file://hsr_meshes/meshes/wrist_v0/wrist_roll.stl; visual mesh filename=file://hsr_meshes/meshes/wrist_v0/wrist_roll.obj

File: robot/hsr_description/robots/hsrb4s.urdf (robot description, URDF)
Before this commit: robot hsrb, 46 links, 45 joints
Links:
- link arm_flex_link: geometry collision mesh filename=file://hsr_meshes/meshes/arm_v0/arm_flex.stl; visual mesh filename=file://hsr_meshes/meshes/arm_v0/arm_flex_light.dae
- link arm_lift_link: geometry collision mesh filename=file://hsr_meshes/meshes/arm_v0/shoulder.stl; visual mesh filename=file://hsr_meshes/meshes/arm_v0/shoulder.dae
- link arm_roll_link: geometry collision mesh filename=file://hsr_meshes/meshes/arm_v0/arm_roll.stl; visual mesh filename=file://hsr_meshes/meshes/arm_v0/arm_roll_light.dae
- link base_link: geometry collision mesh filename=file://hsr_meshes/meshes/base_v2/base.stl; visual mesh filename=file://hsr_meshes/meshes/base_v2/base_light.dae
- link base_range_sensor_link: geometry collision mesh filename=file://hsr_meshes/meshes/sensors/laser.stl; visual mesh filename=file://hsr_meshes/meshes/sensors/laser.dae
- link hand_l_distal_link: geometry collision mesh filename=file://hsr_meshes/meshes/hand_v0/l_distal.stl; visual mesh filename=file://hsr_meshes/meshes/hand_v0/l_distal.stl
- link hand_l_spring_proximal_link: geometry collision mesh filename=file://hsr_meshes/meshes/hand_v0/l_proximal.stl; visual mesh filename=file://hsr_meshes/meshes/hand_v0/l_proximal.stl
- link hand_palm_link: geometry collision mesh filename=file://hsr_meshes/meshes/hand_v0/palm.stl; visual mesh filename=file://hsr_meshes/meshes/hand_v0/palm.stl
- link hand_r_distal_link: geometry collision mesh filename=file://hsr_meshes/meshes/hand_v0/r_distal.stl; visual mesh filename=file://hsr_meshes/meshes/hand_v0/r_distal.stl
- link hand_r_spring_proximal_link: geometry collision mesh filename=file://hsr_meshes/meshes/hand_v0/r_proximal.stl; visual mesh filename=file://hsr_meshes/meshes/hand_v0/r_proximal.stl
- link head_l_stereo_camera_link: geometry visual mesh filename=file://hsr_meshes/meshes/sensors/head_camera.dae
- link head_pan_link: geometry collision mesh filename=file://hsr_meshes/meshes/head_v1/head_pan.stl; visual mesh filename=file://hsr_meshes/meshes/head_v1/head_pan.dae
- link head_r_stereo_camera_link: geometry visual mesh filename=file://hsr_meshes/meshes/sensors/head_camera.dae
- link head_rgbd_sensor_link: geometry collision mesh filename=file://hsr_meshes/meshes/sensors/rgbd.stl; visual mesh filename=file://hsr_meshes/meshes/sensors/rgbd_light.dae
- link head_tilt_link: geometry collision mesh filename=file://hsr_meshes/meshes/head_v1/head.stl; collision mesh filename=file://hsr_meshes/meshes/head_v1/tablet.stl
- link torso_lift_link: geometry collision mesh filename=file://hsr_meshes/meshes/torso_v0/torso.stl; visual mesh filename=file://hsr_meshes/meshes/torso_v0/torso_light.dae
- link wrist_flex_link: geometry collision cylinder length=0.04 radius=0.017; visual cylinder length=0.02 radius=0.017
- link wrist_roll_link: geometry collision mesh filename=file://hsr_meshes/meshes/wrist_v0/wrist_roll.stl; visual mesh filename=file://hsr_meshes/meshes/wrist_v0/wrist_roll.dae
